Commit message: adding packages and generating Manifest.toml file

File: urdf/bravo_5_example.urdf (robot description, URDF)
Before this commit: robot bravo_5_example, 20 links, 19 joints
Links:
- link bravo_1013_base_link: geometry collision cylinder length=0.030 radius=0.046; collision cylinder length=0.1 radius=0.046
- link bravo_1013_joint_link: geometry collision cylinder length=0.03 radius=0.046; visual mesh filename=C:/Users/marcu/OneDrive/Documents/GitHub/onr_compliance_jul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
- link bravo_1019_end_link: geometry visual mesh filename=C:/Users/marcu/OneDrive/Documents/GitHub/onr_compliance_jul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
- link bravo_1023_0_base_link: geometry collision cylinder length=0.03 radius=0.0408; collision cylinder length=0.0816 radius=0.0408
- link bravo_1023_0_joint_link: geometry collision cylinder length=0.080 radius=0.0408; visual mesh filename=C:/Users/marcu/OneDrive/Documents/GitHub/onr_compliance_jul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
- link bravo_1023_1_joint_link: geometry collision cylinder length=0.0056 radius=0.0408; visual mesh filename=C:/Users/marcu/OneDrive/Documents/GitHub/onr_compliance_jul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
- link bravo_1028_base_link: geometry collision cylinder length=0.120 radius=0.0408; visual mesh filename=C:/Users/marcu/OneDrive/Documents/GitHub/onr_compliance_jul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
- link bravo_1030_base_link: geometry collision cylinder length=0.03033333 radius=0.041; collision cylinder length=0.03033333 radius=0.042
- link bravo_base_link: geometry collision box size=0.050 0.080 0.060; collision box size=0.0725 0.1112 0.083
- link bravo_finger_jaws_base_link: geometry collision cylinder length=0.02 radius=0.05; visual mesh filename=C:/Users/marcu/OneDrive/Documents/GitHub/onr_compliance_jul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
- link bravo_finger_jaws_rs2_300_link: geometry collision box size=0.14 0.04 0.045; visual mesh filename=C:/Users/marcu/OneDrive/Documents/GitHub/onr_compliance_jul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
- link bravo_finger_jaws_rs2_301_link: geometry collision box size=0.14 0.04 0.045; visual mesh filename=C:/Users/marcu/OneDrive/Documents/GitHub/onr_compliance_jul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
