Commit message: created bravo_seabotix urdf

File: urdf/bravo_seabotix.urdf (robot description, URDF)
Before this commit: robot bravo_5_example, 20 links, 19 joints
Links:
- added link B_L_bar; visual box size=0.25 0.02 0.05
- added link B_R_bar; visual box size=0.25 0.02 0.05
- added link F_L_bar; visual box size=0.25 0.02 0.05
- added link F_R_bar; visual box size=0.25 0.02 0.05
- added link L_bar; visual box size=0.5 0.02 0.05
- added link R_bar; visual box size=0.5 0.02 0.05
- added link front_bumper; visual cylinder length=0.4 radius=0.075
- added link l_arrow; visual box size=0.05 0.318 0.01
- added link pa_fan; visual cylinder length=0.04 radius=0.06
- added link pa_thruster; visual cylinder length=0.1 radius=0.02
- added link pf_fan; visual cylinder length=0.04 radius=0.06
- added link pf_thruster; visual cylinder length=0.1 radius=0.02
- added link r_arrow; visual box size=0.05 0.318 0.01
- added link rear_bumper; visual cylinder length=0.4 radius=0.075
- added link sa_fan; visual cylinder length=0.04 radius=0.06
- added link sa_thruster; visual cylinder length=0.1 radius=0.02
- added link seabotix_bottle; visual cylinder length=0.26 radius=0.05
- added link sf_fan; visual cylinder length=0.04 radius=0.06
- added link sf_thruster; visual cylinder length=0.1 radius=0.02
- added link vehicle_base_link, mass 30.3; visual box size=0.5 0.4 0.15
Joints:
- added joint BLBarJoint: type fixed, parent vehicle_base_link, child B_L_bar, origin xyz=-0.225 .19 -.2 rpy=0 1.57075 0
- added joint BRBarJoint: type fixed, parent vehicle_base_link, child B_R_bar, origin xyz=-0.225 -.19 -.2 rpy=0 1.57075 0
- added joint FLBarJoint: type fixed, parent vehicle_base_link, child F_L_bar, origin xyz=0.225 .19 -.2 rpy=0 1.57075 0
- added joint FRBarJoint: type fixed, parent vehicle_base_link, child F_R_bar, origin xyz=0.225 -.19 -.2 rpy=0 1.57075 0
- added joint LBarJoint: type fixed, parent vehicle_base_link, child L_bar, origin xyz=0 .19 -.3 rpy=0 0 0
- added joint RBarJoint: type fixed, parent vehicle_base_link, child R_bar, origin xyz=0 -.19 -.3 rpy=0 0 0
- added joint arm_to_vehicle: type fixed, parent vehicle_base_link, child base_link, origin xyz=.325 0 -.09 rpy=3.1415 0 0
- added joint base_to_pa_fan: type fixed, parent vehicle_base_link, child pa_fan, origin xyz=-0.22 0.12 -0.14 rpy=0 -1.57579632679 0.785
- added joint base_to_pf_fan: type fixed, parent vehicle_base_link, child pf_fan, origin xyz=0.22 0.12 -0.14 rpy=0 1.57579632679 -0.785
- added joint base_to_sa_fan: type fixed, parent vehicle_base_link, child sa_fan, origin xyz=-0.22 -0.12 -0.14 rpy=0 -1.57579632679 -0.785
- added joint base_to_sf_fan: type fixed, parent vehicle_base_link, child sf_fan, origin xyz=0.22 -0.12 -0.14 rpy=0 1.57579632679 0.785
- added joint fbump_link: type fixed, parent vehicle_base_link, child front_bumper, origin xyz=0.25 0 0 rpy=1.57579632679 0 0
- added joint l_arrow_link: type fixed, parent vehicle_base_link, child l_arrow, origin xyz=0.05 0.095 0.075 rpy=0 0 0.787898163397
- added joint pa_fan_thruster_joint: type fixed, parent pa_fan, child pa_thruster, origin xyz=0 0 -0.06
- added joint pf_fan_thruster_joint: type fixed, parent pf_fan, child pf_thruster, origin xyz=0 0 -0.06
- added joint r_arrow_link: type fixed, parent vehicle_base_link, child r_arrow, origin xyz=0.05 -0.095 0.075 rpy=0 0 -0.787898163397
- added joint rbump_link: type fixed, parent vehicle_base_link, child rear_bumper, origin xyz=-0.25 0 0 rpy=1.57579632679 0 0
- added joint sa_fan_thruster_joint: type fixed, parent sa_fan, child sa_thruster, origin xyz=0 0 -0.06
- added joint sbottle_link: type fixed, parent vehicle_base_link, child seabotix_bottle, origin xyz=-0.05 0 -0.18 rpy=0 1.57579632679 0
- added joint sf_fan_thruster_joint: type fixed, parent sf_fan, child sf_thruster, origin xyz=0 0 -0.06
