Commit message: remade obj files in Blender and updated bravo5_seabotix urdf

File: urdf/bravo5_seabotix.urdf (robot description, URDF)
Before this commit: robot uvms_alpha_seabotix, 40 links, 39 joints
Links:
- link bravo_jaws_base_link: geometry visual mesh filename=C:/Users/marcu/OneDrive/Documents/GitHub/onr_compliance_jul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
Joints:
- joint bravo_1013_end_joint: origin xyz=0.046 0 -0.05055 rpy=3.14159 0 3.14159 -> xyz=0.046 -0.05055 0.00055 rpy=3.14159 0 0
- joint bravo_1023_0_end_joint: origin xyz=0.0408 0 -0.09385 rpy=3.14159 0 0 -> xyz=0.0408 -0.09385 0 rpy=3.14159 0 0
- joint bravo_1023_1_end_joint: origin xyz=0 0 0.0056 rpy=0 0 0 -> xyz=0 0.0056 0 rpy=0 0 0
- joint bravo_1028_end_joint: origin xyz=0 0 0.120 rpy=-1.5707 -1.5707 0 -> xyz=0 0.120 0 rpy=0 0 1.5707
- joint bravo_axis_b: limit (none) -> lower=0.0 upper=0.0 effort=0 velocity=0
- joint bravo_axis_c: origin xyz=0.042 0 0.0578 rpy=0 0 0 -> xyz=0.042 0.0578 0 rpy=0 0 0
- joint bravo_axis_d: origin xyz=0.046 0 0.0642 rpy=0 0 0 -> xyz=0.046 0.0642 0 rpy=0 0 0
- joint bravo_axis_e: origin xyz=0.0665 0 0.08 rpy=0 0 3.14159 -> xyz=0.0665 0.08 0 rpy=0 0 3.14159
- joint bravo_c_base_joint: origin xyz=0 0 0.182 rpy=0 0 0 -> xyz=0 0.182 0 rpy=0 0 0
- joint bravo_d_base_joint: origin xyz=0 0 0 rpy=0 0 0 -> xyz=0 0 0 rpy=0 0 3.1415
- joint bravo_finger_jaws_rs2_300_joint: origin xyz=0.0097 -0.033 0 rpy=0 0 0 -> xyz=0.0097 0 0.033 rpy=0 0 0
- joint bravo_finger_jaws_rs2_301_joint: origin xyz=0.0097 0.033 0 rpy=0 0 0 -> xyz=0.0097 0 -0.033 rpy=0 0 0
- joint bravo_joint: origin xyz=0 0 0 rpy=0 0 0 -> xyz=0 0 0 rpy=-1.5708 0 0
