Commit message: accessing .obj files locally

File: urdf/bravo7_seabotix.urdf (robot description, URDF)
Before this commit: robot uvms_alpha_seabotix, 32 links, 31 joints
Links:
- link bravo_1013_joint_link: geometry collision cylinder length=0.03 radius=0.0408; collision cylinder length=0.03 radius=0.046
- link bravo_1019_end_link: geometry collision cylinder length=0.03 radius=0.046; collision cylinder length=0.1 radius=0.046
- link bravo_1023_0_joint_link: geometry collision cylinder length=0.08 radius=0.0408; visual mesh filename=C:/Users/marcu/OneDrive/Documents/GitHub/onr_compliance_jul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
- link bravo_1023_1_joint_link: geometry collision cylinder length=0.0056 radius=0.0408; collision cylinder length=0.02 radius=0.05
- link bravo_1026_0_joint_link: geometry collision cylinder length=0.08 radius=0.0408; visual mesh filename=C:/Users/marcu/OneDrive/Documents/GitHub/onr_compliance_jul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
- link bravo_1026_1_joint_link: geometry collision cylinder length=0.0056 radius=0.0408; collision cylinder length=0.03 radius=0.0408
- link bravo_base_link: geometry collision box size=0.05 0.08 0.06; collision box size=0.0725 0.1112 0.083
- link bravo_finger_jaws_rs2_300_link: geometry collision mesh filename=C:/Users/marcu/OneDrive/Documents/GitHub/onr_compliance_jul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; visual mesh filename=C:/Users/marcu/OneDrive/Documents/GitHub/onr_compliance_jul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
- link bravo_finger_jaws_rs2_301_link: geometry collision mesh filename=C:/Users/marcu/OneDrive/Documents/GitHub/onr_compliance_jul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; visual mesh filename=C:/Users/marcu/OneDrive/Documents/GitHub/onr_compliance_jul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
