Commit message: updating src dir

File: urdf/bravo_7.urdf.xacro (robot description, xacro)
@@ -41,5 +41,5 @@
             <visual>
                 <geometry>
-                    <mesh filename="package://bpl_bravo_description_real/meshes/RS2-1019_base.obj" />
+                    <mesh filename="C:/Users/marcu/OneDrive/Documents/GitHub/onr_compliance_julia/meshes/RS2-1019_base.obj" />
                 </geometry>
                 <material name="bravo_black" />
@@ -80,19 +80,19 @@
             <visual>
                 <geometry>
-                    <mesh filename="package://bpl_bravo_description_real/meshes/RS2-1019_end.obj" />
-                </geometry>
-                <material name="bravo_black" />
-                <origin xyz="0.0 0.0 0.0" rpy="0.0 -0.0 0.0" />
-            </visual>
-            <visual>
-                <geometry>
-                    <mesh filename="package://bpl_bravo_description_real/meshes/RS2-1013_base.obj" />
-                </geometry>
-                <material name="bravo_black" />
-                <origin xyz="0.0 0.0 0.0" rpy="0.0 -0.0 0.0" />
-            </visual>
-            <collision>
-                <geometry>
-                    <mesh filename="package://bpl_bravo_description_real/meshes/RS2-1019_end.obj" />
+                    <mesh filename="C:/Users/marcu/OneDrive/Documents/GitHub/onr_compliance_julia/meshes/RS2-1019_end.obj" />
+                </geometry>
+                <material name="bravo_black" />
+                <origin xyz="0.0 0.0 0.0" rpy="0.0 -0.0 0.0" />
+            </visual>
+            <visual>
+                <geometry>
+                    <mesh filename="C:/Users/marcu/OneDrive/Documents/GitHub/onr_compliance_julia/meshes/RS2-1013_base.obj" />
+                </geometry>
+                <material name="bravo_black" />
+                <origin xyz="0.0 0.0 0.0" rpy="0.0 -0.0 0.0" />
+            </visual>
+            <collision>
+                <geometry>
+                    <mesh filename="C:/Users/marcu/OneDrive/Documents/GitHub/onr_compliance_julia/meshes/RS2-1019_end.obj" />
                 </geometry>
                 <origin xyz="0.0 0.0 0.0" rpy="0.0 -0.0 0.0" />
@@ -126,12 +126,12 @@
             <visual>
                 <geometry>
-                    <mesh filename="package://bpl_bravo_description_real/meshes/RS2-1013_end.obj" />
-                </geometry>
-                <material name="bravo_black" />
-                <origin xyz="0.0 0.0 0.0" rpy="0.0 -0.0 0.0" />
-            </visual>
-            <visual>
-                <geometry>
-                    <mesh filename="package://bpl_bravo_description_real/meshes/RS2-1026_0_base.obj" />
+                    <mesh filename="C:/Users/marcu/OneDrive/Documents/GitHub/onr_compliance_julia/meshes/RS2-1013_end.obj" />
+                </geometry>
+                <material name="bravo_black" />
+                <origin xyz="0.0 0.0 0.0" rpy="0.0 -0.0 0.0" />
+            </visual>
+            <visual>
+                <geometry>
+                    <mesh filename="C:/Users/marcu/OneDrive/Documents/GitHub/onr_compliance_julia/meshes/RS2-1026_0_base.obj" />
                 </geometry>
                 <material name="bravo_black" />
@@ -140,5 +140,5 @@
             <visual>
                 <geometry>
-                    <mesh filename="package://bpl_bravo_description_real/meshes/RS2-1030.obj" />
+                    <mesh filename="C:/Users/marcu/OneDrive/Documents/GitHub/onr_compliance_julia/meshes/RS2-1030.obj" />
                 </geometry>
                 <material name="bravo_black" />
@@ -215,5 +215,5 @@
             <visual>
                 <geometry>
-                    <mesh filename="package://bpl_bravo_description_real/meshes/RS2-1026_0_end.obj" />
+                    <mesh filename="C:/Users/marcu/OneDrive/Documents/GitHub/onr_compliance_julia/meshes/RS2-1026_0_end.obj" />
                 </geometry>
                 <material name="bravo_black" />
@@ -242,5 +242,5 @@
             <visual>
                 <geometry>
-                    <mesh filename="package://bpl_bravo_description_real/meshes/RS2-1026_1_end.obj" />
+                    <mesh filename="C:/Users/marcu/OneDrive/Documents/GitHub/onr_compliance_julia/meshes/RS2-1026_1_end.obj" />
                 </geometry>
                 <material name="bravo_black" />
@@ -249,5 +249,5 @@
             <visual>
                 <geometry>
-                    <mesh filename="package://bpl_bravo_description_real/meshes/RS2-1023_0_base.obj" />
+                    <mesh filename="C:/Users/marcu/OneDrive/Documents/GitHub/onr_compliance_julia/meshes/RS2-1023_0_base.obj" />
                 </geometry>
                 <material name="bravo_black" />
@@ -281,5 +281,5 @@
             <visual>
                 <geometry>
-                    <mesh filename="package://bpl_bravo_description_real/meshes/RS2-1023_0_end.obj" />
+                    <mesh filename="C:/Users/marcu/OneDrive/Documents/GitHub/onr_compliance_julia/meshes/RS2-1023_0_end.obj" />
                 </geometry>
                 <material name="bravo_black" />
@@ -308,12 +308,12 @@
             <visual>
                 <geometry>
-                    <mesh filename="package://bpl_bravo_description_real/meshes/RS2-1023_1_end.obj" />
-                </geometry>
-                <material name="bravo_black" />
-                <origin xyz="0.0 0.0 0.0" rpy="0.0 -0.0 0.0" />
-            </visual>
-            <visual>
-                <geometry>
-                    <mesh filename="package://bpl_bravo_description_real/meshes/RS2-1028.obj" />
+                    <mesh filename="C:/Users/marcu/OneDrive/Documents/GitHub/onr_compliance_julia/meshes/RS2-1023_1_end.obj" />
+                </geometry>
+                <material name="bravo_black" />
+                <origin xyz="0.0 0.0 0.0" rpy="0.0 -0.0 0.0" />
+            </visual>
+            <visual>
+                <geometry>
+                    <mesh filename="C:/Users/marcu/OneDrive/Documents/GitHub/onr_compliance_julia/meshes/RS2-1028.obj" />
                 </geometry>
                 <material name="bravo_black" />
@@ -322,5 +322,5 @@
             <visual>
                 <geometry>
-                    <mesh filename="package://bpl_bravo_description_real/meshes/end_effectors/RS2-257.obj" />
+                    <mesh filename="C:/Users/marcu/OneDrive/Documents/GitHub/onr_compliance_julia/meshes/end_effectors/RS2-257.obj" />
                 </geometry>
                 <material name="bravo_finger_jaws_black" />
@@ -361,5 +361,5 @@
             <visual>
                 <geometry>
-                    <mesh filename="package://bpl_bravo_description_real/meshes/end_effectors/RS2-300.obj" />
+                    <mesh filename="C:/Users/marcu/OneDrive/Documents/GitHub/onr_compliance_julia/meshes/end_effectors/RS2-300.obj" />
                 </geometry>
                 <material name="bravo_finger_jaws_black" />
@@ -368,5 +368,5 @@
             <collision>
                 <geometry>
-                    <mesh filename="package://bpl_bravo_description_real/meshes/end_effectors/RS2-300.obj" />
+                    <mesh filename="C:/Users/marcu/OneDrive/Documents/GitHub/onr_compliance_julia/meshes/end_effectors/RS2-300.obj" />
                 </geometry>
                 <origin xyz="0.0 0.0 0.0" rpy="0.0 -0.0 0.0" />
@@ -381,5 +381,5 @@
             <visual>
                 <geometry>
-                    <mesh filename="package://bpl_bravo_description_real/meshes/end_effectors/RS2-301.obj" />
+                    <mesh filename="C:/Users/marcu/OneDrive/Documents/GitHub/onr_compliance_julia/meshes/end_effectors/RS2-301.obj" />
                 </geometry>
                 <material name="bravo_finger_jaws_black" />
@@ -388,5 +388,5 @@
             <collision>
                 <geometry>
-                    <mesh filename="package://bpl_bravo_description_real/meshes/end_effectors/RS2-301.obj" />
+                    <mesh filename="C:/Users/marcu/OneDrive/Documents/GitHub/onr_compliance_julia/meshes/end_effectors/RS2-301.obj" />
                 </geometry>
                 <origin xyz="0.0 0.0 0.0" rpy="0.0 -0.0 0.0" />

File: urdf/bravo_7_example.urdf (robot description, URDF)
Before this commit: robot bravo_7_example, 12 links, 11 joints
Links:
- link bravo_1013_joint_link: geometry collision cylinder length=0.03 radius=0.0408; collision cylinder length=0.03 radius=0.046
- link bravo_1019_end_link: geometry collision cylinder length=0.03 radius=0.046; collision cylinder length=0.1 radius=0.046
- link bravo_1023_0_joint_link: geometry collision cylinder length=0.08 radius=0.0408; visual mesh filename=C:/Users/marcu/OneDrive/Documents/GitHub/onr_compliance_jul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
- link bravo_1023_1_joint_link: geometry collision cylinder length=0.0056 radius=0.0408; collision cylinder length=0.02 radius=0.05
- link bravo_1026_0_joint_link: geometry collision cylinder length=0.08 radius=0.0408; visual mesh filename=C:/Users/marcu/OneDrive/Documents/GitHub/onr_compliance_jul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
- link bravo_1026_1_joint_link: geometry collision cylinder length=0.0056 radius=0.0408; collision cylinder length=0.03 radius=0.0408
- link bravo_base_link: geometry collision box size=0.05 0.08 0.06; collision box size=0.0725 0.1112 0.083
- link bravo_finger_jaws_rs2_300_link: geometry collision mesh filename=C:/Users/marcu/OneDrive/Documents/GitHub/onr_compliance_jul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; visual mesh filename=C:/Users/marcu/OneDrive/Documents/GitHub/onr_compliance_jul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
- link bravo_finger_jaws_rs2_301_link: geometry collision mesh filename=C:/Users/marcu/OneDrive/Documents/GitHub/onr_compliance_jul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; visual mesh filename=C:/Users/marcu/OneDrive/Documents/GitHub/onr_compliance_jul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
