Commit message: added original origins as comments

File: urdf/bravo_7_example.urdf (robot description, URDF)
Before this commit: robot bravo_7_example, 12 links, 11 joints
Joints:
- joint bravo_joint: origin xyz=0 0 0 rpy=1.5708 0 0 -> xyz=0 0 0 rpy=1.5709 0 0

Commit message: orienting joint rotation axes

File: urdf/bravo_7_example.urdf (robot description, URDF)
Before this commit: robot bravo_7_example, 12 links, 11 joints
Joints:
- joint bravo_axis_b: axis  0.  0. -1. ->  0.  -1. 0.
- joint bravo_axis_c: axis  0. -1.  0. ->  0. 0. -1.
- joint bravo_axis_d: axis  0.  0. -1. ->  0.  -1. 0.
- joint bravo_axis_e: axis  0. -1.  0. ->  0. 0.  -1.
- joint bravo_axis_f: axis  0. -1.  0. ->  0. 0. -1.
- joint bravo_axis_g: axis  0.  0. -1. ->  0.  -1. 0.
- joint bravo_finger_jaws_rs2_300_joint: axis  0.  0. -1. ->  0.  -1. 0.
- joint bravo_finger_jaws_rs2_301_joint: axis 0. 0. 1. -> 0. 1. 0.
- joint bravo_joint: origin xyz=0 0 0 rpy=1.5709 0 0 -> xyz=0 0 0 rpy=1.57079 0 0
