Commit message: fixed axis-of-rotation issue

File: urdf/bravo7_test_axis_flop.urdf (robot description, URDF)
Before this commit: robot bravo_7_example, 15 links, 14 joints
Links:
- removed link depth_cam_link
- removed link depth_cam_measurement_link
- removed link kinect_optical_link
- link bravo_1013_joint_link: geometry collision cylinder length=0.03 radius=0.0408; collision cylinder length=0.03 radius=0.046
- link bravo_1019_end_link: geometry collision cylinder length=0.03 radius=0.046; collision cylinder length=0.1 radius=0.046
- link bravo_1023_0_joint_link: geometry collision cylinder length=0.08 radius=0.0408; visual mesh filename=C:/Users/marcu/OneDrive/Documents/GitHub/onr_compliance_jul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
- link bravo_1023_1_joint_link: geometry collision cylinder length=0.0056 radius=0.0408; collision cylinder length=0.02 radius=0.05
- link bravo_1026_0_joint_link: geometry collision cylinder length=0.08 radius=0.0408; visual mesh filename=C:/Users/marcu/OneDrive/Documents/GitHub/onr_compliance_jul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
- link bravo_1026_1_joint_link: geometry collision cylinder length=0.0056 radius=0.0408; collision cylinder length=0.03 radius=0.0408
- link bravo_base_link: geometry collision box size=0.05 0.08 0.06; collision box size=0.0725 0.1112 0.083
- link bravo_finger_jaws_rs2_300_link: geometry collision mesh filename=C:/Users/marcu/OneDrive/Documents/GitHub/onr_compliance_jul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; visual mesh filename=C:/Users/marcu/OneDrive/Documents/GitHub/onr_compliance_jul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
- link bravo_finger_jaws_rs2_301_link: geometry collision mesh filename=C:/Users/marcu/OneDrive/Documents/GitHub/onr_compliance_jul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; visual mesh filename=C:/Users/marcu/OneDrive/Documents/GitHub/onr_compliance_jul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
Joints:
- removed joint depth_cam_measurement
- removed joint depth_cam_to_kinect_optical_link
- removed joint jaw_offset_frame

File: urdf/bravo_7_example.urdf (robot description, URDF)
Before this commit: robot bravo_7_example, 12 links, 11 joints
Joints:
- joint bravo_axis_c: origin xyz=-0.041999999999852135 0.0634 0 rpy=0.0 3.14159 3.14159 -> xyz=-0.041999999999852135 0.058 0.005 rpy=0.0 3.06659 3.14159
- joint bravo_axis_d: origin xyz=0.0408 -0.09434999999999824 0.0056 rpy=3.14159 -0.0 0.0 -> xyz=0.0408 -0.09434999999999824 0.001 rpy=3.14159 0.1 0.0
- joint bravo_axis_e: origin xyz=0 -0.29035 0 rpy=0 0 0 -> xyz=0.0040000000018364235 -0.29034 0 rpy=0 -0.075 0
