Commit message: loading planar bravo to seabotix

File: urdf/bravo7_planar_seabotix.urdf (robot description, URDF)
Before this commit: robot bravo_7_example, 12 links, 11 joints
Links:
- added link B_L_bar; visual box size=0.25 0.02 0.05
- added link B_R_bar; visual box size=0.25 0.02 0.05
- added link F_L_bar; visual box size=0.25 0.02 0.05
- added link F_R_bar; visual box size=0.25 0.02 0.05
- added link L_bar; visual box size=0.5 0.02 0.05
- added link R_bar; visual box size=0.5 0.02 0.05
- added link front_bumper; visual cylinder length=0.4 radius=0.075
- added link l_arrow; visual box size=0.05 0.318 0.01
- added link pa_fan; visual cylinder length=0.04 radius=0.06
- added link pa_thruster; visual cylinder length=0.1 radius=0.02
- added link pf_fan; visual cylinder length=0.04 radius=0.06
- added link pf_thruster; visual cylinder length=0.1 radius=0.02
- added link r_arrow; visual box size=0.05 0.318 0.01
- added link rear_bumper; visual cylinder length=0.4 radius=0.075
- added link sa_fan; visual cylinder length=0.04 radius=0.06
- added link sa_thruster; visual cylinder length=0.1 radius=0.02
- added link seabotix_bottle; visual cylinder length=0.26 radius=0.05
- added link sf_fan; visual cylinder length=0.04 radius=0.06
- added link sf_thruster; visual cylinder length=0.1 radius=0.02
- added link vehicle_base_link, mass 30.3; visual box size=0.5 0.4 0.15
Joints:
- added joint BLBarJoint: type fixed, parent vehicle_base_link, child B_L_bar, origin xyz=-0.225 .19 -.2 rpy=0 1.57075 0
- added joint BRBarJoint: type fixed, parent vehicle_base_link, child B_R_bar, origin xyz=-0.225 -.19 -.2 rpy=0 1.57075 0
- added joint FLBarJoint: type fixed, parent vehicle_base_link, child F_L_bar, origin xyz=0.225 .19 -.2 rpy=0 1.57075 0
- added joint FRBarJoint: type fixed, parent vehicle_base_link, child F_R_bar, origin xyz=0.225 -.19 -.2 rpy=0 1.57075 0
- added joint LBarJoint: type fixed, parent vehicle_base_link, child L_bar, origin xyz=0 .19 -.3 rpy=0 0 0
- added joint RBarJoint: type fixed, parent vehicle_base_link, child R_bar, origin xyz=0 -.19 -.3 rpy=0 0 0
- added joint arm_to_vehicle: type fixed, parent vehicle_base_link, child world, origin xyz=.325 0 -.09 rpy=0 0 0
- added joint base_to_pa_fan: type fixed, parent vehicle_base_link, child pa_fan, origin xyz=-0.22 0.12 -0.14 rpy=0 -1.57579632679 0.785
- added joint base_to_pf_fan: type fixed, parent vehicle_base_link, child pf_fan, origin xyz=0.22 0.12 -0.14 rpy=0 1.57579632679 -0.785
- added joint base_to_sa_fan: type fixed, parent vehicle_base_link, child sa_fan, origin xyz=-0.22 -0.12 -0.14 rpy=0 -1.57579632679 -0.785
- added joint base_to_sf_fan: type fixed, parent vehicle_base_link, child sf_fan, origin xyz=0.22 -0.12 -0.14 rpy=0 1.57579632679 0.785
- added joint fbump_link: type fixed, parent vehicle_base_link, child front_bumper, origin xyz=0.25 0 0 rpy=1.57579632679 0 0
- added joint l_arrow_link: type fixed, parent vehicle_base_link, child l_arrow, origin xyz=0.05 0.095 0.075 rpy=0 0 0.787898163397
- added joint pa_fan_thruster_joint: type fixed, parent pa_fan, child pa_thruster, origin xyz=0 0 -0.06
- added joint pf_fan_thruster_joint: type fixed, parent pf_fan, child pf_thruster, origin xyz=0 0 -0.06
- added joint r_arrow_link: type fixed, parent vehicle_base_link, child r_arrow, origin xyz=0.05 -0.095 0.075 rpy=0 0 -0.787898163397
- added joint rbump_link: type fixed, parent vehicle_base_link, child rear_bumper, origin xyz=-0.25 0 0 rpy=1.57579632679 0 0
- added joint sa_fan_thruster_joint: type fixed, parent sa_fan, child sa_thruster, origin xyz=0 0 -0.06
- added joint sbottle_link: type fixed, parent vehicle_base_link, child seabotix_bottle, origin xyz=-0.05 0 -0.18 rpy=0 1.57579632679 0
- added joint sf_fan_thruster_joint: type fixed, parent sf_fan, child sf_thruster, origin xyz=0 0 -0.06
- joint bravo_axis_a: type prismatic -> fixed
- joint bravo_axis_b: origin xyz=0.0408 -1.326794896676365e-09 -0.09434999999999824 rpy=3.14159 -0.0 0.6 -> xyz=0.0408 -0.09434999999999824 0 rpy=3.14159 -0.0 0; type continuous -> fixed
- joint bravo_axis_c: axis  0. -1.  0. ->  0. 0. -1.; origin xyz=-0.041999999999852135 1.1145077132081467e-07 0.0634 rpy=0.0 -0.0 3.14159 -> xyz=-0.041999999999852135 0.058 0.005 rpy=0.0 3.06659 3.14159
- joint bravo_axis_d: origin xyz=0.0408 -1.326794896676365e-09 -0.09434999999999824 rpy=3.14159 -0.0 0.0 -> xyz=0.0408 -0.09434999999999824 0.001 rpy=3.14159 0.1 0.0; type revolute -> fixed
- joint bravo_axis_e: axis  0. -1.  0. ->  0. 0. -1.; origin xyz=0.0040000000018364235 7.477816037645589e-07 -0.29034999999915573 rpy=3.14159 -0.0 3.14159 -> xyz=0.0040000000018364235 -0.29034 0 rpy=0 -0.075 0
- joint bravo_axis_f: axis  0. -1.  0. ->  0. 0. -1.; origin xyz=0.046 0.0 0.0642 rpy=0.0 -0.0 0.0 -> xyz=-0.046 -0.0642 0 rpy=0.0 -0.0 3.14159
- joint bravo_axis_g: axis  0.  0. -1. ->  0. -1. 0.; origin xyz=0.0665 0.0 0.08 rpy=0.0 0.0 3.14159 -> xyz=0.0665 0.08 0.0 rpy=0.0 0.0 3.14159; type revolute -> fixed
- joint bravo_finger_jaws_rs2_300_joint: origin xyz=-0.032999065323888854 -3.178784226673016e-06 0.1353031787392095 rpy=-1.5707 -1.5706999999997038 0.0 -> xyz=0 0.13529682117078565 -0.033 rpy=0 3.14159 -1.5707; type revolute -> fixed
- joint bravo_finger_jaws_rs2_301_joint: origin xyz=0.03300093406370696 3.178784226673016e-06 0.13529682117078565 rpy=-1.5707 -1.5706999999997038 0.0 -> xyz=0 0.13529682117078565 0.033 rpy=0 3.14159 -1.5707; type revolute -> fixed
- joint bravo_joint: origin xyz=0 0 0 rpy=0 0 0 -> xyz=0 0 0 rpy=1.57079 0 0

Commit message: restructuring URDF

File: urdf/bravo7_planar_seabotix.urdf (robot description, URDF)
Before this commit: robot uvms_alpha_seabotix, 32 links, 31 joints
Links:
- removed link bravo_push_rod
- removed link world
Joints:
- removed joint arm_to_vehicle
- removed joint bravo_axis_a
- joint bravo_joint: origin xyz=0 0 0 rpy=1.57079 0 0 -> xyz=.325 0 -.09 rpy=1.57079 0 0; parent world -> vehicle_base_link

Commit message: fixing coordinate systems transfer between julia and matlab

File: urdf/bravo7_planar_seabotix.urdf (robot description, URDF)
Before this commit: robot uvms_alpha_seabotix, 30 links, 29 joints
Joints:
- joint bravo_axis_c: axis  0. 0. -1. ->  0. 0. 1.; origin xyz=-0.041999999999852135 0.058 0.005 rpy=0.0 3.06659 3.14159 -> xyz=-0.041999999999852135 0.058 0.005 rpy=0.0 3.14159 0
- joint bravo_axis_e: axis  0. 0. -1. ->  0. 0. 1.; origin xyz=0.0040000000018364235 -0.29034 0 rpy=0 -0.075 0 -> xyz=0.0040000000018364235 -0.29034 0 rpy=0 0 3.14159
- joint bravo_axis_f: axis  0. 0. -1. ->  0. 0. 1.

Commit message: need to figure out traj waypoint gen

File: urdf/bravo7_planar_seabotix.urdf (robot description, URDF)
Before this commit: robot uvms_alpha_seabotix, 30 links, 29 joints
Joints:
- joint bravo_axis_c: axis  0. 0. 1. ->  0. 0. -1.
- joint bravo_axis_e: axis  0. 0. 1. ->  0. 0. -1.
- joint bravo_axis_f: axis  0. 0. 1. ->  0. 0. -1.
