Commit message: simplified sim to accomidate fixed arm joints

File: urdf/bravo7_planar_toy_saab copy.urdf (robot description, URDF)
Before this commit: robot bravo_toy_saab, 32 links, 31 joints
Joints:
- joint bravo_axis_c: axis  0. 0. 1. ->  0. 0. -1.; type revolute -> fixed
- joint bravo_axis_e: axis  0. 0. 1. ->  0. 0. -1.; origin xyz=0.0040000000018364235 -0.29034 0 rpy=0 0 3.14159 -> xyz=0.0040000000018364235 -0.29034 0 rpy=0 0 0; type revolute -> fixed
- joint bravo_axis_f: axis  0. 0. 1. ->  0. 0. -1.; origin xyz=-0.046 -0.0642 0 rpy=0.0 -0.0 3.14159 -> xyz=-0.046 -0.0642 0 rpy=0.0 -0.0 -1.57; type revolute -> fixed

Commit message: reorg of simple version

File: urdf/bravo7_planar_toy_saab copy.urdf (robot description, URDF)
Before this commit: robot bravo_toy_saab, 32 links, 31 joints
Joints:
- joint bravo_axis_c: origin xyz=-0.041999999999852135 0.058 0.005 rpy=0.0 3.14159 0 -> xyz=-0.041999999999852135 0.058 0.005 rpy=0.0 3.14159 3.14159
- joint bravo_axis_d: origin xyz=0.0408 -0.09434999999999824 0.001 rpy=3.14159 0.1 0.0 -> xyz=0.0408 -0.09434999999999824 0.001 rpy=3.14159 0.0 0.0
- joint bravo_axis_e: axis  0. 0. -1. ->  0. 0. 1.
- joint bravo_axis_f: origin xyz=-0.046 -0.0642 0 rpy=0.0 -0.0 -1.57 -> xyz=-0.046 -0.0642 0 rpy=0.0 -0.0 -3.14159

Commit message: adding buoyancy balance to simple urdf version

File: urdf/bravo7_planar_toy_saab copy.urdf (robot description, URDF)
Before this commit: robot bravo_toy_saab, 32 links, 31 joints
Links:
- link bravo_1013_joint_link: mass 1.14 -> 0.67141
- link bravo_1019_end_link: mass 1.55 -> 0.95180
- link bravo_1023_0_joint_link: mass 0.333 -> 0.04820
- link bravo_1026_0_joint_link: mass 1.14 -> 0.63153
- link bravo_1026_1_joint_link: mass 1.03 -> 0.60129
- link bravo_base_link: mass 1.25 -> 0.53216
- link bravo_finger_jaws_rs2_300_link: mass 0.24 -> 0.15524
- link bravo_finger_jaws_rs2_301_link: mass 0.24 -> 0.15524
Joints:
- joint bravo_axis_f: origin xyz=-0.046 -0.0642 0 rpy=0.0 -0.0 -3.14159 -> xyz=-0.046 -0.0642 0 rpy=0.0 -0.0 -0
