Commit message: finished urdf regen

File: urdf/arm_vehicle.urdf (robot description, URDF)
Before this commit: robot bravo_toy_saab, 32 links, 31 joints
Links:
- added link new_base
- link bravo_1013_joint_link: mass 1.14 -> 0.67141
- link bravo_1019_end_link: mass 1.55 -> 0.95180
- link bravo_1023_0_joint_link: mass 0.333 -> 0.04820
- link bravo_1023_1_joint_link: mass 1.04 -> 0.56144
- link bravo_1026_0_joint_link: mass 1.14 -> 0.63153
- link bravo_1026_1_joint_link: mass 1.03 -> 0.60129
- link bravo_base_link: mass 1.25 -> 0.53216
- link bravo_finger_jaws_rs2_300_link: mass 0.24 -> 0.15524
- link bravo_finger_jaws_rs2_301_link: mass 0.24 -> 0.15524
Joints:
- added joint planar_world: type revolute, parent new_base, child vehicle_base_link, origin xyz=0 0 0 rpy=0 0 0, axis  0. 1. 0.
- joint bravo_axis_b: origin xyz=0.0408 -0.09434999999999824 0.0 rpy=3.14159 -1.4707 0.0 -> xyz=0.0408 -0.09434999999999824 0.003 rpy=3.14159 -1.5707 0.0
- joint bravo_axis_c: origin xyz=-0.041 -0.058 0.0055 rpy=0 0.1 3.14159 -> xyz=-0.041 -0.058 0.0055 rpy=0 0 0; type revolute -> fixed
- joint bravo_axis_d: origin xyz=0.0408 -0.1 -0.0065 rpy=0.0 0.1 0 -> xyz=0.0408 -0.1 -0.003 rpy=0.0 0.0 0
- joint bravo_axis_e: origin xyz=0.0040000000018364235 -0.289 0.0 rpy=0 0.0 3.14159 -> xyz=0.0040000000018364235 -0.289 0.0 rpy=0 0.0 0; type revolute -> fixed
- joint bravo_axis_f: origin xyz=0.046 0.0642 0.0 rpy=0.0 0.0 0.0 -> xyz=0.046 0.0642 0.0 rpy=0.0 0.0 0; type revolute -> fixed

Commit message: rebuild urdf made better calcs

File: urdf/arm_vehicle.urdf (robot description, URDF)
Before this commit: robot bravo_toy_saab, 33 links, 32 joints
Links:
- link bottom_body_link: mass 30 -> 20
- link vehicle_base_link: mass 30 -> 40
Joints:
- joint bravo_axis_a: axis 0. 0. 1. -> 0. 0. -1.; origin xyz=0.008999999958245167 0.0 0.12560000008350966 rpy=-1.5707 -1.5706999999997038 0.0 -> xyz=0.008999999958245167 0.12560000008350966 0.0 rpy=-1.5707 0.0 1.5706999999997038
- joint bravo_axis_f: origin xyz=0.046 0.0642 0.0 rpy=0.0 0.0 0 -> xyz=0.046 0.0642 0.0 rpy=0.0 0.0 1.5707
- joint ee_link_joint: origin xyz=0 0 0.120 rpy=0 0 -1.5707 -> xyz=0 0.120 0 rpy=0 0 -1.5707
- joint planar_world: origin xyz=0 0 0 rpy=0 0 0 -> xyz=0 0 0.125 rpy=0 0 0

Commit message: refining pitch data collection

File: urdf/arm_vehicle.urdf (robot description, URDF)
Before this commit: robot bravo_toy_saab, 33 links, 32 joints
Joints:
- joint bravo_axis_f: origin xyz=0.046 0.0642 0.0 rpy=0.0 0.0 1.5707 -> xyz=0.046 0.0642 0.0 rpy=0.0 0.0 1.2

Commit message: making linear stiffness estimate

File: urdf/arm_vehicle.urdf (robot description, URDF)
Before this commit: robot bravo_toy_saab, 33 links, 32 joints
Joints:
- joint bravo_axis_c: origin xyz=-0.041 -0.058 0.0055 rpy=0 0 -0.7853981633974483 -> xyz=-0.041 -0.058 0.0055 rpy=0 0 0
- joint bravo_axis_e: origin xyz=0.0040000000018364235 -0.289 0.0 rpy=0 0.0 -0.7853981633974483 -> xyz=0.0040000000018364235 -0.289 0.0 rpy=0 0.0 -0.6416
- joint bravo_axis_f: origin xyz=0.046 0.0642 0.0 rpy=0.0 0.0 2.356194490192345 -> xyz=0.046 0.0642 0.0 rpy=0.0 0.0 1.5707
