Commit message: fixing coordinate frames and making new angle gen and FK

File: test/bravo7_planar.urdf (robot description, URDF)
Before this commit: robot bravo_7_example, 12 links, 11 joints
Links:
- added link end_effector_tip; visual box size=0.0 0.0 0.00
Joints:
- added joint end_effector_tip_joint: type fixed, parent bravo_1023_0_joint_link, child end_effector_tip, origin xyz=0.042 0.0 -0.367 rpy=0.0 3.14159 0.0, axis 0.0 -1 0.0
- joint bravo_axis_a: origin xyz=-8.669411487068951e-07 0.008999999958245167 0.12560000008350966 rpy=-1.5707 -1.5706999999997038 0.0 -> xyz=-8.669411487068951e-07 0.008999999958245167 0.12560000008350966 rpy=-1.5707 -1.5706999999997038 -1.5707
