Commit message: playing with COM calculations

File: test/base_joint.urdf (robot description, URDF)
Before this commit: robot bravo_7_example, 3 links, 2 joints
Links:
- removed link test
- added link bravo_1013_joint_link, mass 1.14; visual mesh filename=package://bpl_bravo_description_real/meshes/RS2-1013_end.stl; visual mesh filename=package://bpl_bravo_description_real/meshes/RS2-1026_0_base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
- added link bravo_1019_end_link, mass 1.55; visual mesh filename=package://bpl_bravo_description_real/meshes/RS2-1013_base.s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; visual mesh filename=package://bpl_bravo_description_real/meshes/RS2-1019_end.stl
Joints:
- removed joint test_joint
- added joint bravo_axis_f: type revolute, parent bravo_1019_end_link, child bravo_1013_joint_link, origin xyz=0.046 0.0 0.0642 rpy=-1.5708 -0.0 0.0, axis  0. -1.  0., limit lower=0.0 upper=3.14 effort=500.0 velocity=3.0
- added joint bravo_axis_g: type fixed, parent bravo_base_link, child bravo_1019_end_link, origin xyz=0.0 0.0 0.039 rpy=0.0 0.0 0, axis  0.  0. -1., limit lower=0.0 upper=6.2 effort=500.0 velocity=3.0
