Commit message: refined downsampling of collision free data

File: test/arm_vehicle.urdf (robot description, URDF)
Before this commit: robot bravo_toy_saab, 33 links, 32 joints
Links:
- added link end_effector_tip; visual box size=0.0 0.0 0.00
- link bravo_1013_joint_link: mass 0.67141 -> 1.14; geometry collision cylinder length=0.03 radius=0.0408; collision cylinder length=0.03 radius=0.046
- link bravo_1019_end_link: mass 0.95180 -> 1.55; geometry collision cylinder length=0.03 radius=0.046; collision cylinder length=0.1 radius=0.046
- link bravo_1023_0_joint_link: mass 0.04820 -> 0.333; geometry collision cylinder length=0.08 radius=0.0408; visual mesh filename=package://bpl_bravo_description_real/meshes/RS2-1023_0_end.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
- link bravo_1023_1_joint_link: mass 0.56144 -> 1.04; geometry collision cylinder length=0.0056 radius=0.0408; collision cylinder length=0.02 radius=0.05
- link bravo_1026_0_joint_link: mass 0.63153 -> 1.14; geometry collision cylinder length=0.08 radius=0.0408; visual mesh filename=package://bpl_bravo_description_real/meshes/RS2-1026_0_end.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
- link bravo_1026_1_joint_link: mass 0.60129 -> 1.03; geometry collision cylinder length=0.0056 radius=0.0408; collision cylinder length=0.03 radius=0.0408
- link bravo_base_link: mass 0.53216 -> 1.25; geometry collision box size=0.05 0.08 0.06; collision box size=0.0725 0.1112 0.083
- link bravo_finger_jaws_rs2_300_link: mass 0.15524 -> 0.24; geometry collision mesh filename=package://bpl_bravo_description_real/meshes/end_effectors/R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; visual mesh filename=package://bpl_bravo_description_real/meshes/end_effectors/R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
- link bravo_finger_jaws_rs2_301_link: mass 0.15524 -> 0.24; geometry collision mesh filename=package://bpl_bravo_description_real/meshes/end_effectors/R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; visual mesh filename=package://bpl_bravo_description_real/meshes/end_effectors/R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
Joints:
- added joint end_effector_tip_joint: type fixed, parent bravo_1023_0_joint_link, child end_effector_tip, origin xyz=0.042 0.0 -0.367 rpy=0.0 3.14159 0.0, axis 0.0 -1 0.0
- joint bravo_axis_a: axis 0. 0. -1. -> 0. 0. 1.; origin xyz=0.008999999958245167 0.12560000008350966 0.0 rpy=-1.5707 0.0 1.5706999999997038 -> xyz=-8.669411487068951e-07 0.008999999958245167 0.12560000008350966 rpy=-1.5707 -1.5706999999997038 -1.5707
- joint bravo_axis_b: origin xyz=0.0408 -0.09434999999999824 0.003 rpy=3.14159 -1.5707 0.0 -> xyz=0.0408 -1.326794896676365e-09 -0.09434999999999824 rpy=3.14159 -0.0 1.5707
- joint bravo_axis_c: axis  0. 0. 1. ->  0. -1.  0.; origin xyz=-0.041 -0.058 0.0055 rpy=0 0 -0.7853981633974483 -> xyz=-0.041999999999852135 1.1145077132081467e-07 0.0634 rpy=0.0 -0.0 3.14159; type fixed -> revolute
- joint bravo_axis_d: axis  0.  0. 1. ->  0.  0. -1.; origin xyz=0.0408 -0.1 -0.003 rpy=0.0 0.0 0 -> xyz=0.0408 -1.326794896676365e-09 -0.09434999999999824 rpy=3.14159 -0.0 0.0
- joint bravo_axis_e: axis  0. 0. 1. ->  0. -1.  0.; origin xyz=0.0040000000018364235 -0.289 0.0 rpy=0 0.0 -0.7853981633974483 -> xyz=0.0040000000018364235 7.477816037645589e-07 -0.29034999999915573 rpy=3.14159 -0.0 3.14159; type fixed -> revolute
- joint bravo_axis_f: axis  0. 0. 1. ->  0. -1.  0.; origin xyz=0.046 0.0642 0.0 rpy=0.0 0.0 2.356194490192345 -> xyz=0.046 0.0 0.0642 rpy=0.0 -0.0 0.0; type fixed -> revolute
- joint bravo_axis_g: origin xyz=0.0665 0.08 0.0 rpy=0.0 0.0 0 -> xyz=0.0665 0.0 0.08 rpy=0.0 0.0 0
- joint bravo_finger_jaws_rs2_300_joint: origin xyz=-0.032999065323888854 0.1353031787392095 0.0 rpy=-1.5707 0.0 1.5707 -> xyz=-0.032999065323888854 -3.178784226673016e-06 0.1353031787392095 rpy=-1.5707 -1.8357 0.0
- joint bravo_finger_jaws_rs2_301_joint: origin xyz=0.03300093406370696 0.13529682117078565 0.0 rpy=-1.5707 0 1.5707 -> xyz=0.03300093406370696 3.178784226673016e-06 0.13529682117078565 rpy=-1.5707 -1.3057 0.0
- joint bravo_joint: origin xyz=.425 0 -.39 rpy=1.57079 0 0 -> xyz=.425 0 -.39 rpy=0 0 0
- joint ee_link_joint: origin xyz=0 0.120 0 rpy=0 0 -1.5707 -> xyz=0 0 0.120 rpy=0 0 -1.5707
- joint planar_world: limit (none) -> lower=0.0 upper=1.0 effort=400.0 velocity=3.0
