Commit message: testing joint/dimension reduction methods

File: test/bravo7.urdf (robot description, URDF)
Before this commit: robot bravo_7_example, 12 links, 11 joints
Joints:
- joint bravo_axis_a: type prismatic -> fixed

Commit message: testing large dataset in .mat file

File: test/bravo7.urdf (robot description, URDF)
Before this commit: robot bravo_7_example, 12 links, 11 joints
Joints:
- joint bravo_finger_jaws_rs2_300_joint: type revolute -> fixed
- joint bravo_finger_jaws_rs2_301_joint: type revolute -> fixed

Commit message: opened jaws till they were not intersecting

File: test/bravo7.urdf (robot description, URDF)
Before this commit: robot bravo_7_example, 12 links, 11 joints
Joints:
- joint bravo_finger_jaws_rs2_300_joint: origin xyz=-0.032999065323888854 -3.178784226673016e-06 0.1353031787392095 rpy=-1.5707 -1.5706999999997038 0.0 -> xyz=-0.032999065323888854 -3.178784226673016e-06 0.1353031787392095 rpy=-1.5707 -1.8357 0.0
- joint bravo_finger_jaws_rs2_301_joint: origin xyz=0.03300093406370696 3.178784226673016e-06 0.13529682117078565 rpy=-1.5707 -1.5706999999997038 0.0 -> xyz=0.03300093406370696 3.178784226673016e-06 0.13529682117078565 rpy=-1.5707 -1.3057 0.0

Commit message: adding in modified urdf and traj planning

File: test/bravo7.urdf (robot description, URDF)
Before this commit: robot bravo_7_example, 15 links, 14 joints
Links:
- removed link depth_cam_link
- removed link depth_cam_measurement_link
- removed link kinect_optical_link
- added link end_effector_tip; visual box size=0.0 0.0 0.00
Joints:
- removed joint depth_cam_measurement
- removed joint depth_cam_to_kinect_optical_link
- removed joint jaw_offset_frame
- added joint end_effector_tip_joint: type fixed, parent bravo_1023_0_joint_link, child end_effector_tip, origin xyz=0.042 0.0 -0.367 rpy=0.0 3.14159 0.0, axis 0.0 -1 0.0
- joint bravo_axis_b: type continuous -> revolute
- joint bravo_finger_jaws_rs2_300_joint: type revolute -> fixed
- joint bravo_finger_jaws_rs2_301_joint: type revolute -> fixed

File: test/bravo7_ft.urdf (robot description, URDF)
Before this commit: robot bravo_7_example, 15 links, 14 joints
Links:
- removed link depth_cam_link
- removed link depth_cam_measurement_link
- removed link kinect_optical_link
- added link ft_sensor_link, mass 0.05; visual cylinder length=0.041275 radius=0.0402
Joints:
- removed joint depth_cam_measurement
- removed joint depth_cam_to_kinect_optical_link
- removed joint jaw_offset_frame
- added joint ft_sensor_joint: type fixed, parent bravo_1023_0_joint_link, child ft_sensor_link, origin xyz=0.0408 -1.326794896676365e-09 -0.115 rpy=3.14159 -0.0 0.6, axis  0.  0. -1., limit lower=0.0 upper=6.2 effort=500.0 velocity=3.0
- joint bravo_axis_b: origin xyz=0.0408 -1.326794896676365e-09 -0.09434999999999824 rpy=3.14159 -0.0 0.6 -> xyz=0 0 0.020 rpy=0 -0.0 0.0; parent bravo_1023_0_joint_link -> ft_sensor_link; type continuous -> revolute

Commit message: hardware results from hinsdale along with data processing

File: test/bravo7.urdf (robot description, URDF)
Before this commit: robot bravo_7_example, 13 links, 12 joints
Joints:
- joint bravo_axis_b: origin xyz=0.0408 -1.326794896676365e-09 -0.09434999999999824 rpy=3.14159 -0.0 0.6 -> xyz=0.0408 -1.326794896676365e-09 -0.09434999999999824 rpy=3.14159 -0.0 1.5707
- joint end_effector_tip_joint: origin xyz=0.042 0.0 -0.367 rpy=0.0 3.14159 0.0 -> xyz=0.042 0.0 -0.358 rpy=0.0 3.14159 0.0
