Commit message: removing PID controller, separting toy from real sim

File: test/urdf/bravo7.urdf (robot description, URDF)
Before this commit: robot bravo_7_example, 12 links, 11 joints
Joints:
- added joint end_effector_tip_joint: type fixed, parent bravo_1023_0_joint_link, child end_effector_tip, origin xyz=0.042 0.0 -0.367 rpy=0.0 3.14159 0.0, axis 0.0 -1 0.0
