Commit message: simulating over varying config urdfs

File: urdf/planar_configs/bravo7_planar_start.urdf (robot description, URDF)
Before this commit: robot bravo_toy_saab, 32 links, 31 joints
Joints:
- joint bravo_axis_c: origin xyz=-0.041999999999852135 0.058 0.005 rpy=0.0 3.14159 -1.57 -> xyz=-0.041999999999852135 0.058 0.005 rpy=0.0 3.14159 3.14159
- joint bravo_axis_f: origin xyz=-0.046 -0.0642 0 rpy=0.0 -0.0 -3.14159 -> xyz=-0.046 -0.0642 0 rpy=0.0 -0.0 -0
